File: 000/Kicad/PIC16F628A_Comparator_Module_000.sch (KiCad schematic (older format))
At the start: 8 parts, among them U1 PIC16f628a

Commit message: Aggiunta label VREF
Connections:
- net VREF: now reaches U1.1 (RA2/AN2/VREF)
Changed lines of the file:
@@
 LIBS:contrib
 LIBS:valves
+LIBS:PIC16F628A_Comparator_Module_000-cache
 EELAYER 25 0
 EELAYER END
@@
 Wire Notes Line
 	750  3150 750  1900
+Text GLabel 2500 2100 0    45   Input ~ 0
+VREF
 $EndSCHEMATC
